Commit message: added robot control mechanics including control with inverse kinematics. need to fix coordinate system from world to robot

File: data/ur5_gripper.urdf (robot description, URDF)
Before this commit: robot ur5, 52 links, 51 joints
Joints:
- joint elbow_joint: limit lower=-3.14159265 upper=3.14159265 effort=150.0 velocity=3.15 -> lower=-3.14159 upper=3.14159 effort=150.0 velocity=3.15
- joint shoulder_lift_joint: limit lower=-3.14159265 upper=-0.9 effort=150.0 velocity=3.15 -> lower=-3.14159 upper=3.14159 effort=150.0 velocity=3.15
- joint shoulder_pan_joint: limit lower=-3.14159265 upper=3.14159265 effort=150.0 velocity=3.15 -> lower=-180 upper=3.14159 effort=150.0 velocity=3.15
- joint wrist_1_joint: limit lower=-3.14159265 upper=3.14159265 effort=28.0 velocity=3.2 -> lower=-3.14159 upper=3.14159 effort=28.0 velocity=3.2
- joint wrist_2_joint: limit lower=-3.14159265 upper=3.14159265 effort=28.0 velocity=3.2 -> lower=-3.14159 upper=3.14159 effort=28.0 velocity=3.2
- joint wrist_3_joint: limit lower=-3.14159265 upper=3.14159265 effort=28.0 velocity=3.2 -> lower=-3.14159 upper=3.14159 effort=28.0 velocity=3.2
